File: KiCad_Files/Keypad/nrf52840-QIAA-aQFN-73.kicad_sch (KiCad schematic)
At the start: 25 parts

Commit message: Added schematic for USB C, per key rgb led, 2 types of jtag connectors, rf connector, rotary encoder, slider, and OLED pins
Parts:
- removed J?: Conn_01x04, symbol Connector_Generic:Conn_01x04
- added C3: 100nF, symbol Device:C
- added J2: Conn_Coaxial, symbol Connector:Conn_Coaxial
- added J3: Pin Header 2x5, 1.27mm, symbol Connector_Generic:Conn_02x05_Counter_Clockwise
- added J4: TC2050-IDC, symbol Connector_Generic:Conn_02x05_Counter_Clockwise
- added R6: 10k, symbol Device:R_US
- added SW2: RESET, symbol Switch:SW_Push
- gave numbers to parts that had none: 24
Connections:
- net VD is gone; now on net VBUS: R7.2
- net GND: now also C3.2, J2.2 (Ext), J3.3 (Pin_3), J4.3 (Pin_3), SW2.2
- net VBUS: no longer C13.1, R7.1, U1.AD2 (VBUS), U1.Y2 (VDDH)
- net VDD: now also C13.1, R7.1, U1.AD2 (VBUS), U1.Y2 (VDDH), J3.1 (Pin_1), J4.1 (Pin_1), R6.2
- net at C17.2, U1.N24 (DEC5): now also C14.2, C15.2, C16.2, C20.1, C22.1, U1.A18 (DEC2), U1.B5 (DEC4), U1.C1 (DEC1), U1.D23 (DEC3), U1.E24 (DEC6)
- net SWDCLK: now reaches U1.AA24 (SWDCLK)
- net SWDCLK: now also J3.4 (Pin_4), J4.4 (Pin_4)
- net SWDIO: now reaches U1.AC24 (SWDIO)
- net SWDIO: now also J3.2 (Pin_2), J4.2 (Pin_2)
- net P0.18/RESET: no longer names the net of U1.AC13 (P0.18/~{RESET})
- net P0.18/RESET: now also C3.1, R6.1, SW2.1
- net RF: no longer names the net of C7.1, C8.1, L1.2
- net RF: now also J2.1 (In)
- new net VDDF: J3.5 (Pin_5), J4.5 (Pin_5)
- no-connect marks 2 -> 12
Other:
- note added: "Bluetooth Antenna Fliter"
- note added: "Bypass Capacitors"
- note added: "High Frequency External Clock"
- note added: "JTAG Debug and Programming Interface"
- note added: "Low Frequency External Clock"
- note added: "NRF52840-AQFN73"
- note added: "VDD Bypass Capacitors"
- moved on the sheet: C10, C11, C12, C13, C14, C15, C16, C17, C18, C19, C20, C21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
